File: seniordesign/flasher/flasher.sch (KiCad schematic (older format))
At the start: 17 parts, among them IC1 ATTINY24-SS, P1 PROG_PINS, P2 GPIO, P3 OUT, Q1 BC847S, Q2 BC847S

Commit message: Fix footprint library tables more
Parts:
- R1, R2, R3, R4, R5, R6, R7, R8, R9: symbol R -> R-RESCUE-flasher

Commit message: Fix flasher; now generates footprints successfully!
Parts:
- P2: footprint Wire_Pads:SolderWirePad_4xInline_1-2mmDrill -> Pin_Headers:Pin_Header_Straight_1x04
- P3: footprint Wire_Pads:SolderWirePad_4xInline_2mmDrill -> Pin_Headers:Pin_Header_Straight_1x04
Changed lines of the file:
@@
 F 0 "#PWR01" H 1500 700 50  0001 C CNN
 F 1 "+5V" H 1500 990 50  0000 C CNN
-F 2 "" H 1500 850 60  0000 C CNN
+F 2 "Wire_Pads:SolderWirePad_single_1-5mmDrill" H 1500 850 60  0001 C CNN
 F 3 "" H 1500 850 60  0000 C CNN
 	1    1500 850
@@
 F 0 "P2" H 5150 2400 50  0000 C CNN
 F 1 "GPIO" V 5250 2150 50  0000 C CNN
-F 2 "Wire_Pads:SolderWirePad_4xInline_1-2mmDrill" H 5150 2150 60  0001 C CNN
+F 2 "Pin_Headers:Pin_Header_Straight_1x04" H 5150 2150 60  0001 C CNN
 F 3 "" H 5150 2150 60  0000 C CNN
 	1    5150 2150
@@
 F 0 "P3" H 5200 3600 50  0000 C CNN
 F 1 "OUT" V 5300 3350 50  0000 C CNN
-F 2 "Wire_Pads:SolderWirePad_4xInline_2mmDrill" H 5200 3350 60  0001 C CNN
+F 2 "Pin_Headers:Pin_Header_Straight_1x04" H 5200 3350 60  0001 C CNN
 F 3 "" H 5200 3350 60  0000 C CNN
 	1    5200 3350
@@
 F 0 "#PWR011" H 1500 1300 30  0001 C CNN
 F 1 "GND" H 1500 1230 30  0001 C CNN
-F 2 "" H 1500 1300 60  0000 C CNN
+F 2 "Wire_Pads:SolderWirePad_single_1-5mmDrill" H 1500 1300 60  0001 C CNN
 F 3 "" H 1500 1300 60  0000 C CNN
 	1    1500 1300
