File: seniordesign/sensors/sensors.sch (KiCad schematic (older format))
At the start: 35 parts, among them CON1 USB-MICRO-B, P1 JTAG_PROG, P2 UART_PROG, P3 ULTRA_FRONT, P4 ULTRA_BACK, SW1 DIPS_04, U1 ADP151AUJZ-3.3-R7, U2 TM4C123GH6PM, U3 RN-42, U4 FGPMMOPA6H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

Commit message: Fix library break, I think?
Parts:
- BT1: symbol Battery -> BATTERY
Connections:
- wire segments 212 -> 210
Other:
- moved on the sheet: R2, R3, R4, R5, R6, R7, R8, R9, SW1, U4

Commit message: Fix everything in sensors except the DIP switch, battery holder, and LED
Parts:
- C1, C3, C4, C9, FB1: footprint (none) -> Capacitors_SMD:C_0805
- C10, C2, C5, C6, C7: footprint (none) -> Capacitors_SMD:C_0603
- C8: footprint (none) -> Capacitors_SMD:R_0805
- CON1: footprint (none) -> Connect:USB_Micro-B
- D1: footprint (none) -> LEDs:LED-1206
- P1: footprint (none) -> Pin_Headers:Pin_Header_Straight_1x06
- P2, P3, P4: footprint (none) -> Pin_Headers:Pin_Header_Straight_1x04
- R1, R10, R3, R4, R5: footprint (none) -> Resistors_SMD:R_0805
- R2, R6, R7, R8, R9: footprint (none) -> Resistors_SMD:R_0603
- U1: footprint (none) -> Housings_SOT-23_SOT-143_TSOT-6:SOT-23-5
- U3: footprint (none) -> custom_footprints:RovingNetworks_RN-42
- U4: footprint (none) -> custom_footprints:GlobalTop-FGPMMOPA6H
- X1: footprint (none) -> Crystals_Oscillators_SMD:crystal_FA238-TSX3225
Changed lines of the file:
@@
 F 0 "U3" H 8600 2850 60  0000 C CNN
 F 1 "RN-42" H 8600 2250 60  0000 C CNN
-F 2 "" H 8600 2250 60  0000 C CNN
+F 2 "custom_footprints:RovingNetworks_RN-42" H 8600 2250 60  0001 C CNN
 F 3 "" H 8600 2250 60  0000 C CNN
 	1    8600 2250
@@
 F 0 "U1" H 2850 1400 60  0000 C CNN
 F 1 "ADP151AUJZ-3.3-R7" H 2850 1700 60  0000 C CNN
-F 2 "" H 2850 1400 60  0000 C CNN
+F 2 "Housings_SOT-23_SOT-143_TSOT-6:SOT-23-5" H 2850 1400 60  0001 C CNN
 F 3 "" H 2850 1400 60  0000 C CNN
 	1    2850 1400
@@
 F 0 "CON1" H 1000 1850 50  0000 C CNN
 F 1 "USB-MICRO-B" H 1150 1150 50  0000 C CNN
-F 2 "" H 1300 1400 50  0000 C CNN
+F 2 "Connect:USB_Micro-B" H 1300 1400 50  0001 C CNN
 F 3 "" H 1300 1400 50  0000 C CNN
 	1    1300 1500
@@
 F 0 "C2" H 3510 1620 50  0000 L CNN
 F 1 "4.7u" H 3510 1470 50  0000 L CNN
-F 2 "" H 3500 1550 60  0000 C CNN
+F 2 "Capacitors_SMD:C_0603" H 3500 1550 60  0001 C CNN
 F 3 "" H 3500 1550 60  0000 C CNN
 	1    3500 1550
@@
 F 0 "C3" H 4010 2270 50  0000 L CNN
 F 1 "0.1u" H 4010 2120 50  0000 L CNN
-F 2 "" H 4000 2200 60  0000 C CNN
+F 2 "Capacitors_SMD:C_0805" H 4000 2200 60  0001 C CNN
 F 3 "" H 4000 2200 60  0000 C CNN
 	1    4000 2200
@@
 F 0 "C1" H 2310 1620 50  0000 L CNN
 F 1 "10u" H 2310 1470 50  0000 L CNN
-F 2 "" H 2300 1550 60  0000 C CNN
+F 2 "Capacitors_SMD:C_0805" H 2300 1550 60  0001 C CNN
 F 3 "" H 2300 1550 60  0000 C CNN
 	1    2300 1550
@@
 F 0 "C4" H 5260 2270 50  0000 L CNN
 F 1 "2.5u" H 5260 2120 50  0000 L CNN
-F 2 "" H 5250 2200 60  0000 C CNN
+F 2 "Capacitors_SMD:C_0805" H 5250 2200 60  0001 C CNN
 F 3 "" H 5250 2200 60  0000 C CNN
 	1    5250 2200
@@
 F 0 "P1" H 700 4650 50  0000 C CNN
 F 1 "JTAG_PROG" V 800 4300 50  0000 C CNN
-F 2 "" H 700 4300 60  0000 C CNN
+F 2 "Pin_Headers:Pin_Header_Straight_1x06" H 700 4300 60  0001 C CNN
 F 3 "" H 700 4300 60  0000 C CNN
 	1    700  4300
@@
 F 0 "R1" V 6930 3700 50  0000 C CNN
 F 1 "4k7" V 6850 3700 50  0000 C CNN
-F 2 "" V 6780 3700 30  0000 C CNN
+F 2 "Resistors_SMD:R_0805" V 6780 3700 30  0001 C CNN
 F 3 "" H 6850 3700 30  0000 C CNN
 	1    6850 3700
@@
 F 0 "C6" H 6860 4220 50  0000 L CNN
 F 1 "2.3u" H 6860 4070 50  0000 L CNN
-F 2 "" H 6850 4150 60  0000 C CNN
+F 2 "Capacitors_SMD:C_0603" H 6850 4150 60  0001 C CNN
 F 3 "" H 6850 4150 60  0000 C CNN
 	1    6850 4150
@@
 F 0 "X1" H 6400 4490 50  0000 C CNN
 F 1 "16.00 MHz" H 6430 4290 50  0000 L CNN
-F 2 "" H 6400 4400 60  0000 C CNN
+F 2 "Crystals_Oscillators_SMD:crystal_FA238-TSX3225" H 6400 4400 60  0001 C CNN
 F 3 "" H 6400 4400 60  0000 C CNN
 	1    6400 4400
@@
 F 0 "C5" H 6710 4820 50  0000 L CNN
 F 1 "9.0p" H 6710 4670 50  0000 L CNN
-F 2 "" H 6700 4750 60  0000 C CNN
+F 2 "Capacitors_SMD:C_0603" H 6700 4750 60  0001 C CNN
 F 3 "" H 6700 4750 60  0000 C CNN
 	1    6700 4750
@@
 F 0 "C7" H 7010 4820 50  0000 L CNN
 F 1 "9.0p" H 7010 4670 50  0000 L CNN
-F 2 "" H 7000 4750 60  0000 C CNN
+F 2 "Capacitors_SMD:C_0603" H 7000 4750 60  0001 C CNN
 F 3 "" H 7000 4750 60  0000 C CNN
 	1    7000 4750
@@
 F 0 "P2" H 800 2950 50  0000 C CNN
 F 1 "UART_PROG" V 900 2700 50  0000 C CNN
-F 2 "" H 800 2700 60  0000 C CNN
+F 2 "Pin_Headers:Pin_Header_Straight_1x04" H 800 2700 60  0001 C CNN
 F 3 "" H 800 2700 60  0000 C CNN
 	1    800  2700
@@
 F 0 "R2" V 7330 2050 50  0000 C CNN
 F 1 "1K" V 7250 2050 50  0000 C CNN
-F 2 "" V 7180 2050 30  0000 C CNN
+F 2 "Resistors_SMD:R_0603" V 7180 2050 30  0001 C CNN
 F 3 "" H 7250 2050 30  0000 C CNN
 	1    7250 2050
@@
 F 0 "C9" H 7410 2870 50  0000 L CNN
 F 1 "0.1u" H 7410 2720 50  0000 L CNN
-F 2 "" H 7400 2800 60  0000 C CNN
+F 2 "Capacitors_SMD:C_0805" H 7400 2800 60  0001 C CNN
 F 3 "" H 7400 2800 60  0000 C CNN
 	1    7400 2800
@@
 F 0 "R6" V 10130 950 50  0000 C CNN
 F 1 "1k" V 10050 950 50  0000 C CNN
-F 2 "" V 9980 950 30  0000 C CNN
+F 2 "Resistors_SMD:R_0603" V 9980 950 30  0001 C CNN
 F 3 "" H 10050 950 30  0000 C CNN
 	1    10050 950
@@
 F 0 "R7" V 10230 950 50  0000 C CNN
 F 1 "1k" V 10150 950 50  0000 C CNN
-F 2 "" V 10080 950 30  0000 C CNN
+F 2 "Resistors_SMD:R_0603" V 10080 950 30  0001 C CNN
 F 3 "" H 10150 950 30  0000 C CNN
 	1    10150 950
@@
 F 0 "R8" V 10330 950 50  0000 C CNN
 F 1 "1k" V 10250 950 50  0000 C CNN
-F 2 "" V 10180 950 30  0000 C CNN
+F 2 "Resistors_SMD:R_0603" V 10180 950 30  0001 C CNN
 F 3 "" H 10250 950 30  0000 C CNN
 	1    10250 950
@@
 F 0 "R9" V 10430 950 50  0000 C CNN
 F 1 "1k" V 10350 950 50  0000 C CNN
-F 2 "" V 10280 950 30  0000 C CNN
+F 2 "Resistors_SMD:R_0603" V 10280 950 30  0001 C CNN
 F 3 "" H 10350 950 30  0000 C CNN
 	1    10350 950
@@
 F 0 "R10" V 10830 1550 50  0000 C CNN
 F 1 "220" V 10750 1550 50  0000 C CNN
-F 2 "" V 10680 1550 30  0000 C CNN
+F 2 "Resistors_SMD:R_0805" V 10680 1550 30  0001 C CNN
 F 3 "" H 10750 1550 30  0000 C CNN
 	1    10750 1550
@@
 F 0 "C8" H 7260 4620 50  0000 L CNN
 F 1 "0.1u" H 7260 4470 50  0000 L CNN
-F 2 "" H 7250 4550 60  0000 C CNN
+F 2 "Capacitors_SMD:R_0805" H 7250 4550 60  0001 C CNN
 F 3 "" H 7250 4550 60  0000 C CNN
 	1    7250 4550
@@
 F 0 "C10" H 7410 5020 50  0000 L CNN
 F 1 "1u" H 7410 4870 50  0000 L CNN
-F 2 "" H 7400 4950 60  0000 C CNN
+F 2 "Capacitors_SMD:C_0603" H 7400 4950 60  0001 C CNN
 F 3 "" H 7400 4950 60  0000 C CNN
 	1    7400 4950
@@
 F 0 "R4" V 8030 4800 50  0000 C CNN
 F 1 "330" V 7950 4800 50  0000 C CNN
-F 2 "" V 7880 4800 30  0000 C CNN
+F 2 "Resistors_SMD:R_0805" V 7880 4800 30  0001 C CNN
 F 3 "" H 7950 4800 30  0000 C CNN
 	1    7950 4800
@@
 F 0 "R5" V 8030 4900 50  0000 C CNN
 F 1 "330" V 7950 4900 50  0000 C CNN
-F 2 "" V 7880 4900 30  0000 C CNN
+F 2 "Resistors_SMD:R_0805" V 7880 4900 30  0001 C CNN
 F 3 "" H 7950 4900 30  0000 C CNN
 	1    7950 4900
@@
 F 0 "R3" V 7930 4050 50  0000 C CNN
 F 1 "330" V 7850 4050 50  0000 C CNN
-F 2 "" V 7780 4050 30  0000 C CNN
+F 2 "Resistors_SMD:R_0805" V 7780 4050 30  0001 C CNN
 F 3 "" H 7850 4050 30  0000 C CNN
 	1    7850 4050
@@
 F 0 "D1" H 7500 4150 50  0000 L CNN
 F 1 "Led_Small" H 7400 3970 50  0000 L CNN
-F 2 "" V 7550 4050 60  0000 C CNN
+F 2 "LEDs:LED-1206" V 7550 4050 60  0001 C CNN
 F 3 "" V 7550 4050 60  0000 C CNN
 	1    7550 4050
@@
 F 0 "FB1" H 7260 3960 50  0000 C CNN
 F 1 "FERRITEBEAD" H 7250 3800 50  0000 C CNN
-F 2 "" H 7250 3850 60  0000 C CNN
+F 2 "Capacitors_SMD:C_0805" H 7250 3850 60  0001 C CNN
 F 3 "" H 7250 3850 60  0000 C CNN
 	1    7250 3850
@@
 F 0 "P3" H 800 5500 50  0000 C CNN
 F 1 "ULTRA_FRONT" V 900 5250 50  0000 C CNN
-F 2 "" H 800 5250 60  0000 C CNN
+F 2 "Pin_Headers:Pin_Header_Straight_1x04" H 800 5250 60  0001 C CNN
 F 3 "" H 800 5250 60  0000 C CNN
 	1    800  5250
@@
 F 0 "P4" H 800 6200 50  0000 C CNN
 F 1 "ULTRA_BACK" V 900 5950 50  0000 C CNN
-F 2 "" H 800 5950 60  0000 C CNN
+F 2 "Pin_Headers:Pin_Header_Straight_1x04" H 800 5950 60  0001 C CNN
 F 3 "" H 800 5950 60  0000 C CNN
 	1    800  5950
@@
 F 0 "U4" H 9100 5100 60  0000 C CNN
 F 1 "FGPMMOPA6H" H 9100 4500 60  0000 C CNN
-F 2 "" H 9100 4500 60  0000 C CNN
+F 2 "custom_footprints:GlobalTop-FGPMMOPA6H" H 9100 4500 60  0001 C CNN
 F 3 "" H 9100 4500 60  0000 C CNN
 	1    9100 4500

Commit message: Fix sensors; footprints are now correct (probably)!
Parts:
- BT1: footprint (none) -> custom_footprints:BAT-HLD-001
- C8: footprint Capacitors_SMD:R_0805 -> Capacitors_SMD:C_0805
- D1: footprint LEDs:LED-1206 -> Capacitors_SMD:C_0805
- D2: footprint (none) -> LEDs:LED-1206
- SW1: footprint (none) -> custom_footprints:SDA04H1BD
- U2: footprint LQFP64 -> Housings_QFP:LQFP-64_10x10mm_Pitch0.5mm
Changed lines of the file:
@@
 F 0 "U2" H 3450 5950 45  0000 C CNN
 F 1 "TM4C123GH6PM" H 5550 2400 45  0000 C CNN
-F 2 "LQFP64" H 4600 4200 35  0000 C CIN
+F 2 "Housings_QFP:LQFP-64_10x10mm_Pitch0.5mm" H 4600 4200 35  0001 C CIN
 F 3 "" H 4600 4900 60  0000 C CNN
 	1    4600 4200
@@
 F 0 "SW1" V 9950 1450 60  0000 C CNN
 F 1 "DIPS_04" V 10450 1450 60  0000 C CNN
-F 2 "" H 10200 1450 60  0000 C CNN
+F 2 "custom_footprints:SDA04H1BD" H 10200 1450 60  0001 C CNN
 F 3 "" H 10200 1450 60  0000 C CNN
 	1    10200 1450
@@
 F 0 "D2" H 10700 1250 50  0000 L CNN
 F 1 "GREEN" H 10600 1070 50  0000 L CNN
-F 2 "" V 10750 1150 60  0000 C CNN
+F 2 "LEDs:LED-1206" V 10750 1150 60  0001 C CNN
 F 3 "" V 10750 1150 60  0000 C CNN
 	1    10750 1150
@@
 F 0 "C8" H 7260 4620 50  0000 L CNN
 F 1 "0.1u" H 7260 4470 50  0000 L CNN
-F 2 "Capacitors_SMD:R_0805" H 7250 4550 60  0001 C CNN
+F 2 "Capacitors_SMD:C_0805" H 7250 4550 60  0001 C CNN
 F 3 "" H 7250 4550 60  0000 C CNN
 	1    7250 4550
@@
 F 0 "BT1" H 7650 5800 50  0000 L CNN
 F 1 "3.7 Li-ion" H 7650 5700 50  0000 L CNN
-F 2 "" V 7550 5790 60  0000 C CNN
+F 2 "custom_footprints:BAT-HLD-001" V 7550 5790 60  0001 C CNN
 F 3 "" V 7550 5790 60  0000 C CNN
 	1    7550 5750
@@
 F 0 "D1" H 7500 4150 50  0000 L CNN
 F 1 "Led_Small" H 7400 3970 50  0000 L CNN
-F 2 "LEDs:LED-1206" V 7550 4050 60  0001 C CNN
+F 2 "Capacitors_SMD:C_0805" V 7550 4050 60  0001 C CNN
 F 3 "" V 7550 4050 60  0000 C CNN
 	1    7550 4050

Commit message: Add proper bypass cap pair for GPS
Parts:
- added C11: 0.01u, Capacitors_SMD:C_0603, symbol C_Small
- C8: value 0.1u -> 1.0u
Connections:
- net GND: now also C11.2
- net at C8.1, FB1.2, U4.1 (VCC): now also C11.1
Changed lines of the file:
@@
 P 7250 4550
 F 0 "C8" H 7260 4620 50  0000 L CNN
-F 1 "0.1u" H 7260 4470 50  0000 L CNN
+F 1 "1.0u" H 7260 4470 50  0000 L CNN
 F 2 "Capacitors_SMD:C_0805" H 7250 4550 60  0001 C CNN
 F 3 "" H 7250 4550 60  0000 C CNN
@@
 L GND #PWR024
 U 1 1 553CA305
-P 7250 4700
-F 0 "#PWR024" H 7250 4450 50  0001 C CNN
-F 1 "GND" H 7250 4550 50  0000 C CNN
-F 2 "" H 7250 4700 60  0000 C CNN
-F 3 "" H 7250 4700 60  0000 C CNN
-	1    7250 4700
+P 7250 4750
+F 0 "#PWR024" H 7250 4500 50  0001 C CNN
+F 1 "GND" H 7250 4600 50  0000 C CNN
+F 2 "" H 7250 4750 60  0000 C CNN
+F 3 "" H 7250 4750 60  0000 C CNN
+	1    7250 4750
 	1    0    0    -1
 $EndComp
@@
 Connection ~ 6850 3450
 Wire Wire Line
-	7250 4700 7250 4650
+	7250 4750 7250 4650
 Connection ~ 7250 4400
 Connection ~ 2600 2550
@@
 Wire Wire Line
 	7850 3700 7850 3800
+$Comp
+L C_Small C11
+U 1 1 55DBCB69
+P 7450 4550
+F 0 "C11" H 7460 4620 50  0000 L CNN
+F 1 "0.01u" H 7460 4470 50  0000 L CNN
+F 2 "Capacitors_SMD:C_0603" H 7450 4550 60  0001 C CNN
+F 3 "" H 7450 4550 60  0000 C CNN
+	1    7450 4550
+	1    0    0    -1
+$EndComp
+Wire Wire Line
+	7450 4650 7450 4700
+Wire Wire Line
+	7450 4700 7250 4700
+Connection ~ 7250 4700
+Wire Wire Line
+	7450 4450 7450 4400
+Connection ~ 7450 4400
 $EndSCHEMATC

Commit message: Add pushbutton to program TM4C123[...]
Parts:
- added R11: 10k, Resistors_SMD:R_0805, symbol R
- added SW2: SW_PUSH, custom_footprints:1571634-1, symbol SW_PUSH
Connections:
- net GND: now also SW2.2
- net at C2.1, C3.1, C9.1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: now also R11.1
- net at U2.5 (PF4/T2CCP0): now also R11.2, SW2.1

Commit message: Add sensor PCB Gerber files
Connections:
- net at C1.1, CON1.1 (VBUS), U1.1 (VIN)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: now also U1.3 (EN)
Changed lines of the file:
@@
 $EndComp
 $Comp
-L GND #PWR8
+L GND #PWR01
 U 1 1 553BA8B8
 P 2850 1950
-F 0 "#PWR8" H 2850 1700 50  0001 C CNN
+F 0 "#PWR01" H 2850 1700 50  0001 C CNN
 F 1 "GND" H 2850 1800 50  0000 C CNN
 F 2 "" H 2850 1950 60  0000 C CNN
@@
 $EndComp
 $Comp
-L GND #PWR1
+L GND #PWR02
 U 1 1 553BA8DA
 P 700 1850
-F 0 "#PWR1" H 700 1600 50  0001 C CNN
+F 0 "#PWR02" H 700 1600 50  0001 C CNN
 F 1 "GND" H 700 1700 50  0000 C CNN
 F 2 "" H 700 1850 60  0000 C CNN
@@
 $EndComp
 $Comp
-L GND #PWR7
+L GND #PWR03
 U 1 1 553BD6B0
 P 2300 1750
-F 0 "#PWR7" H 2300 1500 50  0001 C CNN
+F 0 "#PWR03" H 2300 1500 50  0001 C CNN
 F 1 "GND" H 2300 1600 50  0000 C CNN
 F 2 "" H 2300 1750 60  0000 C CNN
@@
 $EndComp
 $Comp
-L GND #PWR9
+L GND #PWR04
 U 1 1 553BD6D5
 P 3500 1750
-F 0 "#PWR9" H 3500 1500 50  0001 C CNN
+F 0 "#PWR04" H 3500 1500 50  0001 C CNN
 F 1 "GND" H 3500 1600 50  0000 C CNN
 F 2 "" H 3500 1750 60  0000 C CNN
@@
 $EndComp
 $Comp
-L GND #PWR10
+L GND #PWR05
 U 1 1 553BD6FA
 P 4000 2350
-F 0 "#PWR10" H 4000 2100 50  0001 C CNN
+F 0 "#PWR05" H 4000 2100 50  0001 C CNN
 F 1 "GND" H 4000 2200 50  0000 C CNN
 F 2 "" H 4000 2350 60  0000 C CNN
@@
 $EndComp
 $Comp
-L GND #PWR14
+L GND #PWR06
 U 1 1 553BD71F
 P 5250 2350
-F 0 "#PWR14" H 5250 2100 50  0001 C CNN
+F 0 "#PWR06" H 5250 2100 50  0001 C CNN
 F 1 "GND" H 5250 2200 50  0000 C CNN
 F 2 "" H 5250 2350 60  0000 C CNN
@@
 $EndComp
 $Comp
-L GND #PWR6
+L GND #PWR07
 U 1 1 553BD78E
 P 1950 1800
-F 0 "#PWR6" H 1950 1550 50  0001 C CNN
+F 0 "#PWR07" H 1950 1550 50  0001 C CNN
 F 1 "GND" H 1950 1650 50  0000 C CNN
 F 2 "" H 1950 1800 60  0000 C CNN
@@
 $EndComp
 $Comp
-L GND #PWR11
+L GND #PWR08
 U 1 1 553BDD43
 P 4400 6250
-F 0 "#PWR11" H 4400 6000 50  0001 C CNN
+F 0 "#PWR08" H 4400 6000 50  0001 C CNN
 F 1 "GND" H 4400 6100 50  0000 C CNN
 F 2 "" H 4400 6250 60  0000 C CNN
@@
 $EndComp
 $Comp
-L GND #PWR12
+L GND #PWR09
 U 1 1 553BDD6F
 P 4750 6250
-F 0 "#PWR12" H 4750 6000 50  0001 C CNN
+F 0 "#PWR09" H 4750 6000 50  0001 C CNN
 F 1 "GND" H 4750 6100 50  0000 C CNN
 F 2 "" H 4750 6250 60  0000 C CNN
@@
 $EndComp
 $Comp
-L GND #PWR13
+L GND #PWR010
 U 1 1 553BDD94
 P 5100 6250
-F 0 "#PWR13" H 5100 6000 50  0001 C CNN
+F 0 "#PWR010" H 5100 6000 50  0001 C CNN
 F 1 "GND" H 5100 6100 50  0000 C CNN
 F 2 "" H 5100 6250 60  0000 C CNN
@@
 $EndComp
 $Comp
-L GND #PWR2
+L GND #PWR011
 U 1 1 553BFACB
 P 1000 4650
-F 0 "#PWR2" H 1000 4400 50  0001 C CNN
+F 0 "#PWR011" H 1000 4400 50  0001 C CNN
 F 1 "GND" H 1000 4500 50  0000 C CNN
 F 2 "" H 1000 4650 60  0000 C CNN
@@
 $EndComp
 $Comp
-L GND #PWR18
+L GND #PWR012
 U 1 1 553BFE28
 P 6850 4400
-F 0 "#PWR18" H 6850 4150 50  0001 C CNN
+F 0 "#PWR012" H 6850 4150 50  0001 C CNN
 F 1 "GND" H 6850 4250 50  0000 C CNN
 F 2 "" H 6850 4400 60  0000 C CNN
@@
 $EndComp
 $Comp
-L GND #PWR16
+L GND #PWR013
 U 1 1 553C1E97
 P 6400 4600
-F 0 "#PWR16" H 6400 4350 50  0001 C CNN
+F 0 "#PWR013" H 6400 4350 50  0001 C CNN
 F 1 "GND" H 6400 4450 50  0000 C CNN
 F 2 "" H 6400 4600 60  0000 C CNN
@@
 $EndComp
 $Comp
-L GND #PWR19
+L GND #PWR014
 U 1 1 553C24FA
 P 6900 5000
-F 0 "#PWR19" H 6900 4750 50  0001 C CNN
+F 0 "#PWR014" H 6900 4750 50  0001 C CNN
 F 1 "GND" H 6900 4850 50  0000 C CNN
 F 2 "" H 6900 5000 60  0000 C CNN
@@
 $EndComp
 $Comp
-L GND #PWR29
+L GND #PWR015
 U 1 1 553C2A40
 P 9000 5700
-F 0 "#PWR29" H 9000 5450 50  0001 C CNN
+F 0 "#PWR015" H 9000 5450 50  0001 C CNN
 F 1 "GND" H 9000 5550 50  0000 C CNN
 F 2 "" H 9000 5700 60  0000 C CNN
@@
 $EndComp
 $Comp
-L GND #PWR15
+L GND #PWR016
 U 1 1 553C330C
 P 6250 4700
-F 0 "#PWR15" H 6250 4450 50  0001 C CNN
+F 0 "#PWR016" H 6250 4450 50  0001 C CNN
 F 1 "GND" H 6250 4550 50  0000 C CNN
 F 2 "" H 6250 4700 60  0000 C CNN
@@
 $EndComp
 $Comp
-L GND #PWR27
+L GND #PWR017
 U 1 1 553C3C6E
 P 8300 3500
-F 0 "#PWR27" H 8300 3250 50  0001 C CNN
+F 0 "#PWR017" H 8300 3250 50  0001 C CNN
 F 1 "GND" H 8300 3350 50  0000 C CNN
 F 2 "" H 8300 3500 60  0000 C CNN
@@
 $EndComp
 $Comp
-L GND #PWR28
+L GND #PWR018
 U 1 1 553C3C9E
 P 8800 3500
-F 0 "#PWR28" H 8800 3250 50  0001 C CNN
+F 0 "#PWR018" H 8800 3250 50  0001 C CNN
 F 1 "GND" H 8800 3350 50  0000 C CNN
 F 2 "" H 8800 3500 60  0000 C CNN
@@
 $EndComp
 $Comp
-L GND #PWR24
+L GND #PWR019
 U 1 1 553C3CC7
 P 7550 2850
-F 0 "#PWR24" H 7550 2600 50  0001 C CNN
+F 0 "#PWR019" H 7550 2600 50  0001 C CNN
 F 1 "GND" H 7550 2700 50  0000 C CNN
 F 2 "" H 7550 2850 60  0000 C CNN
@@
 $EndComp
 $Comp
-L GND #PWR23
+L GND #PWR020
 U 1 1 553C3CF0
 P 7450 1700
-F 0 "#PWR23" H 7450 1450 50  0001 C CNN
+F 0 "#PWR020" H 7450 1450 50  0001 C CNN
 F 1 "GND" H 7450 1550 50  0000 C CNN
 F 2 "" H 7450 1700 60  0000 C CNN
@@
 $EndComp
 $Comp
-L GND #PWR3
+L GND #PWR021
 U 1 1 553C4D2C
 P 1100 2900
-F 0 "#PWR3" H 1100 2650 50  0001 C CNN
+F 0 "#PWR021" H 1100 2650 50  0001 C CNN
 F 1 "GND" H 1100 2750 50  0000 C CNN
 F 2 "" H 1100 2900 60  0000 C CNN
@@
 $EndComp
 $Comp
-L GND #PWR30
+L GND #PWR022
 U 1 1 553C6473
 P 10000 2650
-F 0 "#PWR30" H 10000 2400 50  0001 C CNN
+F 0 "#PWR022" H 10000 2400 50  0001 C CNN
 F 1 "GND" H 10000 2500 50  0000 C CNN
 F 2 "" H 10000 2650 60  0000 C CNN
@@
 $EndComp
 $Comp
-L GND #PWR21
+L GND #PWR023
 U 1 1 553C7B41
 P 7400 3000
-F 0 "#PWR21" H 7400 2750 50  0001 C CNN
+F 0 "#PWR023" H 7400 2750 50  0001 C CNN
 F 1 "GND" H 7400 2850 50  0000 C CNN
 F 2 "" H 7400 3000 60  0000 C CNN
@@
 $EndComp
 $Comp
-L GND #PWR20
+L GND #PWR024
 U 1 1 553CA305
 P 7250 4750
-F 0 "#PWR20" H 7250 4500 50  0001 C CNN
+F 0 "#PWR024" H 7250 4500 50  0001 C CNN
 F 1 "GND" H 7250 4600 50  0000 C CNN
 F 2 "" H 7250 4750 60  0000 C CNN
@@
 $EndComp
 $Comp
-L GND #PWR22
+L GND #PWR025
 U 1 1 553CCC74
 P 7400 5150
-F 0 "#PWR22" H 7400 4900 50  0001 C CNN
+F 0 "#PWR025" H 7400 4900 50  0001 C CNN
 F 1 "GND" H 7400 5000 50  0000 C CNN
 F 2 "" H 7400 5150 60  0000 C CNN
@@
 $EndComp
 $Comp
-L GND #PWR26
+L GND #PWR026
 U 1 1 553CD097
 P 7550 6150
-F 0 "#PWR26" H 7550 5900 50  0001 C CNN
+F 0 "#PWR026" H 7550 5900 50  0001 C CNN
 F 1 "GND" H 7550 6000 50  0000 C CNN
 F 2 "" H 7550 6150 60  0000 C CNN
@@
 $EndComp
 $Comp
-L GND #PWR25
+L GND #PWR027
 U 1 1 553CF281
 P 7550 4250
-F 0 "#PWR25" H 7550 4000 50  0001 C CNN
+F 0 "#PWR027" H 7550 4000 50  0001 C CNN
 F 1 "GND" H 7550 4100 50  0000 C CNN
 F 2 "" H 7550 4250 60  0000 C CNN
@@
 $EndComp
 $Comp
-L GND #PWR4
+L GND #PWR028
 U 1 1 553D307D
 P 1100 5500
-F 0 "#PWR4" H 1100 5250 50  0001 C CNN
+F 0 "#PWR028" H 1100 5250 50  0001 C CNN
 F 1 "GND" H 1100 5350 50  0000 C CNN
 F 2 "" H 1100 5500 60  0000 C CNN
@@
 $EndComp
 $Comp
-L GND #PWR5
+L GND #PWR029
 U 1 1 553D31CE
 P 1100 6250
-F 0 "#PWR5" H 1100 6000 50  0001 C CNN
+F 0 "#PWR029" H 1100 6000 50  0001 C CNN
 F 1 "GND" H 1100 6100 50  0000 C CNN
 F 2 "" H 1100 6250 60  0000 C CNN
@@
 Connection ~ 6550 3100
 $Comp
-L GND #PWR17
+L GND #PWR030
 U 1 1 55DCE8F0
 P 6550 3850
-F 0 "#PWR17" H 6550 3600 50  0001 C CNN
+F 0 "#PWR030" H 6550 3600 50  0001 C CNN
 F 1 "GND" H 6550 3700 50  0000 C CNN
 F 2 "" H 6550 3850 60  0000 C CNN
@@
 Wire Wire Line
 	6550 3750 6550 3850
+Wire Wire Line
+	2500 1550 2450 1550
+Wire Wire Line
+	2450 1550 2450 1350
+Connection ~ 2450 1350
 $EndSCHEMATC
